File: feeder/pcb/mobo/mobo.sch (KiCad schematic (older format))
At the start: 25 parts, among them J1 SERIAL_BRIDGE, J2 Spring_Finger_Interface, J3 AVR-ISP-6, M1 Motor_DC, SW1 SW_Push, SW2 SW_Push, SW3 SW_Push, SW4 SW_SPDT, U1 ATmega328-AU, U2 VCNT2020, U3 DRV8838, Y1 Resonator_Small

Commit message: init kicad-exports to auto generate ibom and gerbers
Parts:
- C1: symbol Device:CP1_Small -> mobo-rescue:CP1_Small-Device
- J3: symbol Connector:AVR-ISP-6 -> mobo-rescue:AVR-ISP-6-Connector
- JP1: symbol Device:Jumper_NO_Small -> mobo-rescue:Jumper_NO_Small-Device
- U1: symbol MCU_Microchip_ATmega:ATmega328-AU -> mobo-rescue:ATmega328-AU-MCU_Microchip_ATmega
- U2: symbol stephen:VCNT2020 -> mobo-rescue:VCNT2020-stephen
- U3: symbol stephen:DRV8838 -> mobo-rescue:DRV8838-stephen
Changed lines of the file:
@@
 $EndDescr
 $Comp
-L MCU_Microchip_ATmega:ATmega328-AU U1
+L mobo-rescue:ATmega328-AU-MCU_Microchip_ATmega U1
 U 1 1 5DC9E191
 P 3600 2600
@@
 $EndComp
 $Comp
-L Connector:AVR-ISP-6 J3
+L mobo-rescue:AVR-ISP-6-Connector J3
 U 1 1 5DC9EF1D
 P 1050 2400
@@
 $EndComp
 $Comp
-L Device:CP1_Small C1
+L mobo-rescue:CP1_Small-Device C1
 U 1 1 5DC9F2AC
 P 2550 2350
@@
 	2400 1450 2400 1400
 $Comp
-L stephen:VCNT2020 U2
+L mobo-rescue:VCNT2020-stephen U2
 U 1 1 5DEA2AE3
 P 2450 7050
@@
 $EndComp
 $Comp
-L stephen:DRV8838 U3
+L mobo-rescue:DRV8838-stephen U3
 U 1 1 5E357164
 P 9050 1800
@@
 nSLEEP
 $Comp
-L Device:Jumper_NO_Small JP1
+L mobo-rescue:Jumper_NO_Small-Device JP1
 U 1 1 5E3B5CCA
 P 4700 7200
