File: pnp/pcb/mobo/motor_control.sch (KiCad schematic (older format))
At the start: 37 parts, among them J1 X_MOTOR, J2 Y_MOTOR1, J3 Z_MOTOR, J37 P_MOTOR, J38 C_MOTOR, J4 R_MOTOR, J48 Y_MOTOR2

Commit message: init kicad-exports to auto generate ibom and gerbers
Parts:
- C1, C2, C3, C4, C5, C6: symbol Device:CP -> mobo-rescue:CP-Device
- JP1, JP2, JP22, JP23, JP24, JP25, JP26, JP27, JP28, JP29, JP3, JP30, JP4, JP5, JP6, JP7, JP8, JP9: symbol Device:Jumper_NO_Small -> mobo-rescue:Jumper_NO_Small-Device
Changed lines of the file:
@@
 $EndComp
 $Comp
-L Device:Jumper_NO_Small JP9
+L mobo-rescue:Jumper_NO_Small-Device JP9
 U 1 1 5E406CE8
 P 1350 6950
@@
 $EndComp
 $Comp
-L Device:Jumper_NO_Small JP8
+L mobo-rescue:Jumper_NO_Small-Device JP8
 U 1 1 5E41359A
 P 1350 6850
@@
 $EndComp
 $Comp
-L Device:Jumper_NO_Small JP7
+L mobo-rescue:Jumper_NO_Small-Device JP7
 U 1 1 5E413783
 P 1350 6750
@@
 $EndComp
 $Comp
-L Device:Jumper_NO_Small JP3
+L mobo-rescue:Jumper_NO_Small-Device JP3
 U 1 1 5E418FB7
 P 1450 2650
@@
 $EndComp
 $Comp
-L Device:Jumper_NO_Small JP2
+L mobo-rescue:Jumper_NO_Small-Device JP2
 U 1 1 5E418FDE
 P 1450 2550
@@
 $EndComp
 $Comp
-L Device:Jumper_NO_Small JP1
+L mobo-rescue:Jumper_NO_Small-Device JP1
 U 1 1 5E418FE8
 P 1450 2450
@@
 $EndComp
 $Comp
-L Device:Jumper_NO_Small JP6
+L mobo-rescue:Jumper_NO_Small-Device JP6
 U 1 1 5E421DFB
 P 1000 4900
@@
 $EndComp
 $Comp
-L Device:Jumper_NO_Small JP5
+L mobo-rescue:Jumper_NO_Small-Device JP5
 U 1 1 5E421E22
 P 1000 4800
@@
 $EndComp
 $Comp
-L Device:Jumper_NO_Small JP4
+L mobo-rescue:Jumper_NO_Small-Device JP4
 U 1 1 5E421E2C
 P 1000 4700
@@
 $EndComp
 $Comp
-L Device:CP C1
+L mobo-rescue:CP-Device C1
 U 1 1 5E4332EA
 P 750 900
@@
 $EndComp
 $Comp
-L Device:CP C2
+L mobo-rescue:CP-Device C2
 U 1 1 5E4399B6
 P 1150 900
@@
 $EndComp
 $Comp
-L Device:CP C3
+L mobo-rescue:CP-Device C3
 U 1 1 5E43CEF6
 P 1550 900
@@
 $EndComp
 $Comp
-L Device:Jumper_NO_Small JP30
+L mobo-rescue:Jumper_NO_Small-Device JP30
 U 1 1 5EB0D862
 P 4350 6950
@@
 $EndComp
 $Comp
-L Device:Jumper_NO_Small JP29
+L mobo-rescue:Jumper_NO_Small-Device JP29
 U 1 1 5EB0D889
 P 4350 6850
@@
 $EndComp
 $Comp
-L Device:Jumper_NO_Small JP28
+L mobo-rescue:Jumper_NO_Small-Device JP28
 U 1 1 5EB0D893
 P 4350 6750
@@
 $EndComp
 $Comp
-L Device:Jumper_NO_Small JP24
+L mobo-rescue:Jumper_NO_Small-Device JP24
 U 1 1 5EB0D8BE
 P 4350 2700
@@
 $EndComp
 $Comp
-L Device:Jumper_NO_Small JP23
+L mobo-rescue:Jumper_NO_Small-Device JP23
 U 1 1 5EB0D8E5
 P 4350 2600
@@
 $EndComp
 $Comp
-L Device:Jumper_NO_Small JP22
+L mobo-rescue:Jumper_NO_Small-Device JP22
 U 1 1 5EB0D8EF
 P 4350 2500
@@
 $EndComp
 $Comp
-L Device:Jumper_NO_Small JP27
+L mobo-rescue:Jumper_NO_Small-Device JP27
 U 1 1 5EB0D91A
 P 4500 4900
@@
 $EndComp
 $Comp
-L Device:Jumper_NO_Small JP26
+L mobo-rescue:Jumper_NO_Small-Device JP26
 U 1 1 5EB0D941
 P 4500 4800
@@
 $EndComp
 $Comp
-L Device:Jumper_NO_Small JP25
+L mobo-rescue:Jumper_NO_Small-Device JP25
 U 1 1 5EB0D94B
 P 4500 4700
@@
 NoConn ~ 4850 1700
 $Comp
-L Device:CP C4
+L mobo-rescue:CP-Device C4
 U 1 1 5EB78194
 P 2650 900
@@
 $EndComp
 $Comp
-L Device:CP C5
+L mobo-rescue:CP-Device C5
 U 1 1 5EB781A6
 P 3050 900
@@
 $EndComp
 $Comp
-L Device:CP C6
+L mobo-rescue:CP-Device C6
 U 1 1 5EB781AC
 P 3450 900
