File: pnp/pcb/mobo/power.sch (KiCad schematic (older format))
At the start: 26 parts, among them J45 Jack-DC, U5 AP1117-33, U7 TPS54336ADDA

Commit message: init kicad-exports to auto generate ibom and gerbers
Parts:
- C13, C30, C7: symbol Device:CP -> mobo-rescue:CP-Device
Changed lines of the file:
@@
 $EndComp
 $Comp
-L Device:CP C7
+L mobo-rescue:CP-Device C7
 U 1 1 5EB1E64F
 P 2050 1400
@@
 	4750 1300 4850 1300
 $Comp
-L Device:CP C13
+L mobo-rescue:CP-Device C13
 U 1 1 5EB31705
 P 6800 1650
@@
 	4600 3500 4750 3500
 $Comp
-L Device:CP C30
+L mobo-rescue:CP-Device C30
 U 1 1 5F115598
 P 5200 3650
