File: pnp/pcb/piggyback/feederComm.sch (KiCad schematic (older format))
At the start: 60 parts, among them J10 F06, J11 F07, J12 F08, J13 F09, J14 F10, J15 F11, J16 F12, J17 F13, J18 F14, J19 F15, J20 F16, J21 F17, J22 F18, J23 F19, J24 F20, J25 F25, J26 F26, J27 F27, J28 F28, J29 F21, J30 F22, J31 F23, J32 F24, J33 F29, J34 F30, J35 F31, J36 F32, J5 F01, J6 F02, J7 F03, J8 F04, J9 F05, U1 MCP23017_SO_2, U3 MCP23017_SO_3, U4 MCP23017_SO_1, U5 MCP23017_SO_4

Commit message: init kicad-exports to auto generate ibom and gerbers
Parts:
- JP10, JP11, JP12, JP13, JP14, JP15, JP16, JP17, JP18, JP19, JP20, JP21: symbol Device:Jumper_NO_Small -> piggyback-rescue:Jumper_NO_Small-Device
Changed lines of the file:
@@
 $EndComp
 $Comp
-L Device:Jumper_NO_Small JP10
+L piggyback-rescue:Jumper_NO_Small-Device JP10
 U 1 1 5E46A459
 P 1100 2600
@@
 $EndComp
 $Comp
-L Device:Jumper_NO_Small JP11
+L piggyback-rescue:Jumper_NO_Small-Device JP11
 U 1 1 5E46B27E
 P 1200 2600
@@
 $EndComp
 $Comp
-L Device:Jumper_NO_Small JP12
+L piggyback-rescue:Jumper_NO_Small-Device JP12
 U 1 1 5E46B564
 P 1300 2600
@@
 $EndComp
 $Comp
-L Device:Jumper_NO_Small JP13
+L piggyback-rescue:Jumper_NO_Small-Device JP13
 U 1 1 5E4803DD
 P 1100 5450
@@
 $EndComp
 $Comp
-L Device:Jumper_NO_Small JP14
+L piggyback-rescue:Jumper_NO_Small-Device JP14
 U 1 1 5E4803E3
 P 1200 5450
@@
 $EndComp
 $Comp
-L Device:Jumper_NO_Small JP15
+L piggyback-rescue:Jumper_NO_Small-Device JP15
 U 1 1 5E4803E9
 P 1300 5450
@@
 $EndComp
 $Comp
-L Device:Jumper_NO_Small JP16
+L piggyback-rescue:Jumper_NO_Small-Device JP16
 U 1 1 5E486B50
 P 3850 2650
@@
 $EndComp
 $Comp
-L Device:Jumper_NO_Small JP18
+L piggyback-rescue:Jumper_NO_Small-Device JP18
 U 1 1 5E486B56
 P 3950 2650
@@
 $EndComp
 $Comp
-L Device:Jumper_NO_Small JP20
+L piggyback-rescue:Jumper_NO_Small-Device JP20
 U 1 1 5E486B5C
 P 4050 2650
@@
 $EndComp
 $Comp
-L Device:Jumper_NO_Small JP17
+L piggyback-rescue:Jumper_NO_Small-Device JP17
 U 1 1 5E48D97B
 P 3850 5450
@@
 $EndComp
 $Comp
-L Device:Jumper_NO_Small JP19
+L piggyback-rescue:Jumper_NO_Small-Device JP19
 U 1 1 5E48D981
 P 3950 5450
@@
 $EndComp
 $Comp
-L Device:Jumper_NO_Small JP21
+L piggyback-rescue:Jumper_NO_Small-Device JP21
 U 1 1 5E48D987
 P 4050 5450
