File: pnp/pcb/piggyback/motorControl.sch (KiCad schematic (older format))
At the start: 18 parts, among them J1 STEPPER_1, J2 STEPPER_2, J3 STEPPER_3

Commit message: init kicad-exports to auto generate ibom and gerbers
Parts:
- C1, C2, C3: symbol Device:CP -> piggyback-rescue:CP-Device
- JP1, JP2, JP3, JP4, JP5, JP6, JP7, JP8, JP9: symbol Device:Jumper_NO_Small -> piggyback-rescue:Jumper_NO_Small-Device
Changed lines of the file:
@@
 $EndComp
 $Comp
-L Device:Jumper_NO_Small JP9
+L piggyback-rescue:Jumper_NO_Small-Device JP9
 U 1 1 5E406CE8
 P 1650 6450
@@
 $EndComp
 $Comp
-L Device:Jumper_NO_Small JP8
+L piggyback-rescue:Jumper_NO_Small-Device JP8
 U 1 1 5E41359A
 P 1650 6350
@@
 $EndComp
 $Comp
-L Device:Jumper_NO_Small JP7
+L piggyback-rescue:Jumper_NO_Small-Device JP7
 U 1 1 5E413783
 P 1650 6250
@@
 $EndComp
 $Comp
-L Device:Jumper_NO_Small JP3
+L piggyback-rescue:Jumper_NO_Small-Device JP3
 U 1 1 5E418FB7
 P 1650 2650
@@
 $EndComp
 $Comp
-L Device:Jumper_NO_Small JP2
+L piggyback-rescue:Jumper_NO_Small-Device JP2
 U 1 1 5E418FDE
 P 1650 2550
@@
 $EndComp
 $Comp
-L Device:Jumper_NO_Small JP1
+L piggyback-rescue:Jumper_NO_Small-Device JP1
 U 1 1 5E418FE8
 P 1650 2450
@@
 $EndComp
 $Comp
-L Device:Jumper_NO_Small JP6
+L piggyback-rescue:Jumper_NO_Small-Device JP6
 U 1 1 5E421DFB
 P 1650 4550
@@
 $EndComp
 $Comp
-L Device:Jumper_NO_Small JP5
+L piggyback-rescue:Jumper_NO_Small-Device JP5
 U 1 1 5E421E22
 P 1650 4450
@@
 $EndComp
 $Comp
-L Device:Jumper_NO_Small JP4
+L piggyback-rescue:Jumper_NO_Small-Device JP4
 U 1 1 5E421E2C
 P 1650 4350
@@
 $EndComp
 $Comp
-L Device:CP C1
+L piggyback-rescue:CP-Device C1
 U 1 1 5E4332EA
 P 800 1000
@@
 $EndComp
 $Comp
-L Device:CP C2
+L piggyback-rescue:CP-Device C2
 U 1 1 5E4399B6
 P 1200 1000
@@
 $EndComp
 $Comp
-L Device:CP C3
+L piggyback-rescue:CP-Device C3
 U 1 1 5E43CEF6
 P 1600 1000
