File: pnp/pcb/piggyback/piggyback.sch (KiCad schematic (older format))
At the start: 16 parts, among them J37 Screw_Terminal_01x03, J38 AVR-ISP-6, J39 SERIAL_INTERFACE, J4 USB_B_Micro, SW1 SW_Push_Dual, U2 ATmega32U4-AU, Y1 16MHz

Commit message: init kicad-exports to auto generate ibom and gerbers
Parts:
- J38: symbol Connector:AVR-ISP-6 -> piggyback-rescue:AVR-ISP-6-Connector
- J4: symbol Connector:USB_B_Micro -> piggyback-rescue:USB_B_Micro-Connector
- U2: symbol MCU_Microchip_ATmega:ATmega32U4-AU -> piggyback-rescue:ATmega32U4-AU-MCU_Microchip_ATmega
Changed lines of the file:
@@
 $EndDescr
 $Comp
-L MCU_Microchip_ATmega:ATmega32U4-AU U2
+L piggyback-rescue:ATmega32U4-AU-MCU_Microchip_ATmega U2
 U 1 1 5E3E9AF4
 P 5500 3650
@@
 Contains main uC, comms to computer, all button interfaces and status LEDs
 $Comp
-L Connector:USB_B_Micro J4
+L piggyback-rescue:USB_B_Micro-Connector J4
 U 1 1 5E44822F
 P 4000 3150
@@
 STEPPER_3_DIR
 $Comp
-L Connector:AVR-ISP-6 J38
+L piggyback-rescue:AVR-ISP-6-Connector J38
 U 1 1 5E434974
 P 2300 3250
